File: cad/analyzer_pcb_without_IC.kicad_pcb (KiCad board)
At the start: 2 copper layers, 58.4 x 58.4 mm, 19 parts, among them J1 Conn_Coaxial, J2 Conn_Coaxial, Q1 MMBT3904

Commit message: updated lmh1980 pcb
Parts:
- moved C3 7.18 mm to (83.8, 76.2)
- moved R2 6.35 mm to (86.4, 71.1)
- moved C4 3.59 mm to (81.3, 71.1)
- moved C5 2.54 mm to (71.1, 71.1)
Routing:
- net VCC: track 86.8 -> 36.3 mm, vias 2 -> 3
- net GND: track 117.5 -> 137.2 mm, vias 4 -> 5
- net Net-(R2-Pad2): track 4.19 -> 11.8 mm
- net Net-(R4-Pad1): track 24.2 -> 26.5 mm
- net Net-(R10-Pad1): track 20.6 -> 22.6 mm
- net Net-(C5-Pad2): track 11.3 -> 12.4 mm
- net Net-(R8-Pad1): track 18.9 -> 18.4 mm
